Commit message: hexapod_gazebo_description

File: src/hexapod_gazebo_description/urdf/hexapod_gazebo_3_joint.xacro (robot description, xacro)
@@ -7,21 +7,18 @@
   <xacro:property name="bodymass" value="3"/>
   <xacro:property name="bridgelength" value="0.01"/>
-  <xacro:property name="bridgeradius" value="0.03"/>
+  <xacro:property name="bridgeradius" value="0.02"/>
   <xacro:property name="bridgemass" value="0.5"/>
-  <xacro:property name="rolllength" value="0.093"/>
+  <xacro:property name="rolllength" value="0.14489"/>
   <xacro:property name="rollradius" value="0.03"/>
   <xacro:property name="rollmass" value="${rolllength*5}"/>
-  <xacro:property name="pitch1length" value="0.14489"/>
+  <xacro:property name="pitch1length" value="0.164"/>
   <xacro:property name="pitch1radius" value="0.03"/>
   <xacro:property name="pitch1mass" value="${pitch1length*5}"/>
-  <xacro:property name="pitch2length" value="0.164"/>
+  <xacro:property name="pitch2length" value="0.157"/>
   <xacro:property name="pitch2radius" value="0.03"/>
   <xacro:property name="pitch2mass" value="${pitch2length*5}"/>
-  <xacro:property name="pitch3length" value="0.157"/>
-  <xacro:property name="pitch3radius" value="0.03"/>
-  <xacro:property name="pitch3mass" value="${pitch3length*5}"/>
   <xacro:property name="sticklength" value="0.01"/>
-  <xacro:property name="stickradius" value="0.1"/>
-  <xacro:property name="stickmass" value="1"/>
+  <xacro:property name="stickradius" value="0.08"/>
+  <xacro:property name="stickmass" value="0.5"/>
   <xacro:property name="damping" value="1"/>
 <link name="base_link">
@@ -41,6 +38,6 @@
      <cylinder length="${bodylength}" radius="${bodyradius}"/>
    </geometry>
-   <material name="Red">
-     <color rgba="255 0 0 100"/>
+   <material name="black">
+     <color rgba="0 0 0 100"/>
    </material>
   </visual>
@@ -76,10 +73,10 @@
       <cylinder length="${bridgelength}" radius="${bridgeradius}"/>
     </geometry>
-    <material name="Black">
-      <color rgba="0 0 0 1"/>
+    <material name="white">
+      <color rgba="255 255 255 1"/>
     </material>
   </visual>
   <inertial>
-    <origin xyz="0 0 0" rpy="0 0 0"/>
+    <origin xyz="${bridgelength/2} 0 0" rpy="0 ${M_PI/2} 0"/>
       <mass value="${bridgemass}"/>
       <inertia
@@ -110,10 +107,10 @@
       <cylinder length="${rolllength}" radius="${rollradius}"/>
     </geometry>
-    <material name="Black">
-      <color rgba="0 0 0 1"/>
+    <material name="blue">
+      <color rgba="0 0 255 1"/>
     </material>
   </visual>
   <inertial>
-    <origin xyz="0 0 0" rpy="0 0 0"/>
+    <origin xyz="${rolllength/2} 0 0" rpy="0 ${M_PI/2} 0"/>
       <mass value="${rollmass}"/>
       <inertia
@@ -138,5 +135,5 @@
   <parent link="${leg}_bridge"/>
   <child link="${leg}_roll"/>
-  <origin rpy="0 0 0" xyz="0 0 0"/>
+  <origin rpy="0 0 0" xyz="${bridgelength} 0 0"/>
 </joint>
 <link name="${leg}_pitch1">
@@ -146,10 +143,10 @@
       <cylinder length="${pitch1length}" radius="${pitch1radius}"/>
     </geometry>
-    <material name="Red">
-      <color rgba="255 0 0 1"/>
+    <material name="green">
+      <color rgba="0 128 0 1"/>
     </material>
   </visual>
  <inertial>
-    <origin xyz="0 0 0" rpy="0 0 0"/>
+    <origin xyz="${pitch1length/2} 0 0" rpy="0 ${M_PI/2} 0"/>
       <mass value="${pitch1mass}"/>
       <inertia
@@ -187,5 +184,5 @@
   </visual>
  <inertial>
-    <origin xyz="${pitch2length} 0 0" rpy="0 0 0"/>
+    <origin xyz="${pitch2length/2} 0 0" rpy="${M_PI/2} 0 ${M_PI/2}"/>
       <mass value="${pitch2mass}"/>
       <inertia
@@ -214,42 +211,4 @@
   <origin rpy="0 0 -${M_PI/2}" xyz="${pitch1length} 0 0"/>
 </joint>
-<link name="${leg}_pitch3">
-  <visual>
-    <origin xyz="${pitch3length/2} 0 0" rpy="${M_PI/2} 0 ${M_PI/2}"/>
-    <geometry>
-      <cylinder length="${pitch3length}" radius="${pitch3radius}"/>
-    </geometry>
-    <material name="Red">
-      <color rgba="255 0 0 1"/>
-    </material>
-  </visual>
- <inertial>
-    <origin xyz="0 0 0" rpy="0 0 0"/>
-      <mass value="${pitch3mass}"/>
-      <inertia
-        ixx="${0.5*pitch3mass*pitch3radius*pitch3radius}" ixy="0.0" ixz="0.0"
-        iyy="${(3*pitch3mass*pitch3radius*pitch3radius+4*pitch3mass*pitch3length*pitch3length)/12}" iyz="0.0"
-        izz="${(3*pitch3mass*pitch3radius*pitch3radius+4*pitch3mass*pitch3length*pitch3length)/12}"/>
-    </inertial>
-  <collision>
-    <origin xyz="${pitch3length/2} 0 0" rpy="${M_PI/2} 0 ${M_PI/2}"/>
-    <geometry>
-      <cylinder length="${pitch3length}" radius="${pitch3radius}"/>
-    </geometry>
-  </collision>
-</link>
-  <gazebo reference="${leg}_pitch3">
-    <material>Gazebo/Red</material>
-    <mu1 value="200"/>
-    <mu2 value="200"/>
-  </gazebo>
-<joint name="${leg}_pitch3" type="revolute">
-  <axis xyz="0 0 1"/>
-  <limit effort="300" lower="-${M_PI/3}" upper="${M_PI/2}" velocity="1"/>
-  <dynamics damping="${damping}"/>
-  <parent link="${leg}_pitch2"/>
-  <child link="${leg}_pitch3"/>
-  <origin rpy="0 0 0" xyz="${pitch2length} 0 0"/>
-</joint>
 <!--stick-->
 <link name="${leg}_stick1">
@@ -279,8 +238,8 @@
 </link>
 <joint name="${leg}_stick1" type="revolute">
-  <limit effort="300" lower="-${M_PI/7}" upper="${M_PI/7}" velocity="1"/>
-  <dynamics damping="${damping}"/>
-  <axis xyz="1 0 0"/>
-  <parent link="${leg}_pitch3"/>
+  <limit effort="300" lower="-${M_PI/2}" upper="${M_PI/2}" velocity="1"/>
+  <dynamics damping="${damping}"/>
+  <axis xyz="0 0 1"/>
+  <parent link="${leg}_pitch2"/>
   <child link="${leg}_stick1"/>
   <origin rpy="0 ${M_PI/2} 0" xyz="${pitch2length+sticklength/2} 0 0"/>
@@ -288,15 +247,15 @@
   <gazebo reference="${leg}_stick1">
     <material>Gazebo/Black</material>
-    <mu1 value="10000"/>
-    <mu2 value="10000"/>
-  </gazebo>
-<link name="${leg}_stick3">
-  <visual>
-    <origin xyz="0 0 0" rpy="0 0 0"/>
-    <geometry>
-      <cylinder length="${sticklength}" radius="${stickradius}"/>
-    </geometry>
-    <material name="Black">
-      <color rgba="0 0 0 1"/>
+    <mu1 value="10"/>
+    <mu2 value="10"/>
+  </gazebo>
+<link name="${leg}_stick2">
+  <visual>
+    <origin xyz="0 0 0" rpy="0 0 0"/>
+    <geometry>
+      <cylinder length="0.01" radius="0.01"/>
+    </geometry>
+    <material name="yellow">
+      <color rgba="255 255 0 1"/>
     </material>
   </visual>
@@ -312,29 +271,29 @@
     <origin xyz="0 0 0" rpy="0 0 0"/>
     <geometry>
+      <cylinder length="0.01" radius="0.01"/>
+    </geometry>
+  </collision>
+</link>
+<joint name="${leg}_stick2" type="revolute">
+  <limit effort="300" lower="-${M_PI/2}" upper="${M_PI/2}" velocity="1"/>
+  <dynamics damping="${damping}"/>
+  <axis xyz="1 0 0"/>
+  <parent link="${leg}_stick1"/>
+  <child link="${leg}_stick2"/>
+  <origin rpy="0 0 0" xyz="0 0 0"/>
+</joint>
+  <gazebo reference="${leg}_stick2">
+    <material>Gazebo/Black</material>
+    <mu1 value="10"/>
+    <mu2 value="10"/>
+  </gazebo>
+<link name="${leg}_stick3">
+  <visual>
+    <origin xyz="0 0 0" rpy="0 0 0"/>
+    <geometry>
       <cylinder length="${sticklength}" radius="${stickradius}"/>
     </geometry>
-  </collision>
-</link>
-<joint name="${leg}_stick3" type="revolute">
-  <limit effort="300" lower="-${M_PI/7}" upper="${M_PI/7}" velocity="1"/>
-  <dynamics damping="${damping}"/>
-  <axis xyz="0 1 0"/>
-  <parent link="${leg}_stick1"/>
-  <child link="${leg}_stick3"/>
-  <origin rpy="0 0 0" xyz="0 0 0"/>
-</joint>
-  <gazebo reference="${leg}_stick3">
-    <material>Gazebo/Black</material>
-    <mu1 value="10000"/>
-    <mu2 value="10000"/>
-  </gazebo>
-<!--<link name="${leg}_stick3">
-  <visual>
-    <origin xyz="0 0 0" rpy="0 0 0"/>
-    <geometry>
-      <cylinder length="${sticklength}" radius="${stickradius}"/>
-    </geometry>
-    <material name="Black">
-      <color rgba="0 0 0 1"/>
+    <material name="yellow">
+      <color rgba="255 255 0 1"/>
     </material>
   </visual>
@@ -355,5 +314,5 @@
 </link>
 <joint name="${leg}_stick3" type="revolute">
-  <limit effort="300" lower="-${M_PI/7}" upper="${M_PI/7}" velocity="1"/>
+  <limit effort="300" lower="-${M_PI/2}" upper="${M_PI/2}" velocity="1"/>
   <dynamics damping="${damping}"/>
   <axis xyz="0 1 0"/>
@@ -364,7 +323,7 @@
   <gazebo reference="${leg}_stick3">
     <material>Gazebo/Black</material>
-    <mu1 value="100000"/>
-    <mu2 value="100000"/>
-  </gazebo>-->
+    <mu1 value="0"/>
+    <mu2 value="0"/>
+  </gazebo>
 <!--motor-->
 <transmission name="${leg}_tran1">
@@ -375,5 +334,5 @@
     <actuator name="${leg}_motor1">
       <hardwareInterface>EffortJointInterface</hardwareInterface>
-      <mechanicalReduction>1</mechanicalReduction>
+      <mechanicalReduction>80</mechanicalReduction>
     </actuator>
   </transmission>
@@ -385,5 +344,5 @@
     <actuator name="${leg}_motor2">
       <hardwareInterface>EffortJointInterface</hardwareInterface>
-      <mechanicalReduction>1</mechanicalReduction>
+      <mechanicalReduction>80</mechanicalReduction>
     </actuator>
   </transmission>
@@ -395,25 +354,25 @@
     <actuator name="${leg}_motor3">
       <hardwareInterface>EffortJointInterface</hardwareInterface>
-      <mechanicalReduction>1</mechanicalReduction>
+      <mechanicalReduction>80</mechanicalReduction>
     </actuator>
   </transmission>
 <transmission name="${leg}_tran4">
     <type>transmission_interface/SimpleTransmission</type>
-    <joint name="${leg}_pitch3">
-      <hardwareInterface>EffortJointInterface</hardwareInterface>
-    </joint>
-    <actuator name="${leg}_motor4">
-      <hardwareInterface>EffortJointInterface</hardwareInterface>
-      <mechanicalReduction>1</mechanicalReduction>
+    <joint name="${leg}_stick1">
+      <hardwareInterface>EffortJointInterface</hardwareInterface>
+    </joint>
+    <actuator name="${leg}_stick1">
+      <hardwareInterface>EffortJointInterface</hardwareInterface>
+      <mechanicalReduction>80</mechanicalReduction>
     </actuator>
   </transmission>
 <transmission name="${leg}_tran5">
     <type>transmission_interface/SimpleTransmission</type>
-    <joint name="${leg}_stick1">
-      <hardwareInterface>EffortJointInterface</hardwareInterface>
-    </joint>
-    <actuator name="${leg}_motor5">
-      <hardwareInterface>EffortJointInterface</hardwareInterface>
-      <mechanicalReduction>1</mechanicalReduction>
+    <joint name="${leg}_stick2">
+      <hardwareInterface>EffortJointInterface</hardwareInterface>
+    </joint>
+    <actuator name="${leg}_stick2">
+      <hardwareInterface>EffortJointInterface</hardwareInterface>
+      <mechanicalReduction>80</mechanicalReduction>
     </actuator>
   </transmission>
@@ -423,22 +382,12 @@
       <hardwareInterface>EffortJointInterface</hardwareInterface>
     </joint>
-    <actuator name="${leg}_motor6">
-      <hardwareInterface>EffortJointInterface</hardwareInterface>
-      <mechanicalReduction>1</mechanicalReduction>
-    </actuator>
-  </transmission>
-<!--<transmission name="${leg}_tran7">
-    <type>transmission_interface/SimpleTransmission</type>
-    <joint name="${leg}_stick3">
-      <hardwareInterface>EffortJointInterface</hardwareInterface>
-    </joint>
-    <actuator name="${leg}_motor7">
-      <hardwareInterface>EffortJointInterface</hardwareInterface>
-      <mechanicalReduction>1</mechanicalReduction>
-    </actuator>
-  </transmission>-->
+    <actuator name="${leg}_stick3">
+      <hardwareInterface>EffortJointInterface</hardwareInterface>
+      <mechanicalReduction>80</mechanicalReduction>
+    </actuator>
+  </transmission>
   <gazebo>
      <plugin name="joint_state_publisher" filename="libgazebo_ros_joint_state_publisher.so">
-       <jointName>${leg}_roll, ${leg}_pitch1, ${leg}_pitch2,${leg}_pitch3, ${leg}_stick1, ${leg}_stick3</jointName>
+       <jointName>${leg}_roll, ${leg}_pitch1, ${leg}_pitch2</jointName>
      </plugin>
   </gazebo>
@@ -452,6 +401,6 @@
 <xacro:leg leg="leg2" r="0" p="0" ry="${M_PI/2}" x="0" y="${bodyradius}"/>
 <xacro:leg leg="leg3" r="0" p="0" ry="${M_PI/6*5}" x="-${bodyradius/2*gen3}" y="${bodyradius/2}"/>
-<xacro:leg leg="leg4" r="0" p="0" ry="-${M_PI/6*5}" x="-${bodyradius/2*gen3}" y="-${bodyradius/2}"/>
+<xacro:leg leg="leg6" r="0" p="0" ry="-${M_PI/6*5}" x="-${bodyradius/2*gen3}" y="-${bodyradius/2}"/>
 <xacro:leg leg="leg5" r="0" p="0" ry="-${M_PI/2}" x="0" y="-${bodyradius}"/>
-<xacro:leg leg="leg6" r="0" p="0" ry="-${M_PI/6}" x="${bodyradius/2*gen3}" y="-${bodyradius/2}"/>
+<xacro:leg leg="leg4" r="0" p="0" ry="-${M_PI/6}" x="${bodyradius/2*gen3}" y="-${bodyradius/2}"/>
 </robot>

File: src/hexapod_gazebo_description/urdf/未命名文件夹/hexapod_gazebo.xacro (robot description, xacro)
@@ -6,7 +6,4 @@
   <xacro:property name="bodylength" value="0.1000"/>
   <xacro:property name="bodymass" value="3"/>
-  <xacro:property name="bridgelength" value="0.01"/>
-  <xacro:property name="bridgeradius" value="0.03"/>
-  <xacro:property name="bridgemass" value="0.5"/>
   <xacro:property name="rolllength" value="0.093"/>
   <xacro:property name="rollradius" value="0.03"/>
@@ -70,38 +67,4 @@
 </joint>
   <xacro:macro name="leg" params="leg r p ry x y">
-<link name="${leg}_bridge">
-  <visual>
-    <origin xyz="${bridgelength/2} 0 0" rpy="0 ${M_PI/2} 0"/>
-    <geometry>
-      <cylinder length="${bridgelength}" radius="${bridgeradius}"/>
-    </geometry>
-    <material name="Black">
-      <color rgba="0 0 0 1"/>
-    </material>
-  </visual>
-  <inertial>
-    <origin xyz="0 0 0" rpy="0 0 0"/>
-      <mass value="${bridgemass}"/>
-      <inertia
-        ixx="0" ixy="0.0" ixz="0.0"
-        iyy="0" iyz="0.0"
-        izz="0"/>
-    </inertial>
-  <collision>
-    <origin xyz="${bridgelength/2} 0 0" rpy="0 ${M_PI/2} 0"/>
-    <geometry>
-      <cylinder length="${bridgelength}" radius="${bridgeradius}"/>
-    </geometry>
-  </collision>
-</link>
-  <gazebo reference="${leg}_bridge">
-    <material>Gazebo/Black</material>
-  </gazebo>
-<joint name="${leg}_bridge" type="fixed">
-  <axis xyz="0 0 1"/>
-  <parent link="body"/>
-  <child link="${leg}_bridge"/>
-  <origin rpy="${r} ${p} ${ry}" xyz="${x} ${y} 0"/>
-</joint>
 <link name="${leg}_roll">
   <visual>
@@ -136,7 +99,7 @@
   <limit effort="300" lower="-${M_PI/4}" upper="${M_PI/4}" velocity="1"/>
   <dynamics damping="${damping}"/>
-  <parent link="${leg}_bridge"/>
+  <parent link="body"/>
   <child link="${leg}_roll"/>
-  <origin rpy="0 0 0" xyz="0 0 0"/>
+  <origin rpy="${r} ${p} ${ry}" xyz="${x} ${y} 0"/>
 </joint>
 <link name="${leg}_pitch1">
@@ -440,5 +403,5 @@
   <gazebo>
      <plugin name="joint_state_publisher" filename="libgazebo_ros_joint_state_publisher.so">
-       <jointName>${leg}_roll, ${leg}_pitch1, ${leg}_pitch2,${leg}_pitch3, ${leg}_stick1, ${leg}_stick3</jointName>
+       <jointName>${leg}_roll, ${leg}_pitch1, ${leg}_pitch2,${leg}_pitch3</jointName>
      </plugin>
   </gazebo>
@@ -452,6 +415,6 @@
 <xacro:leg leg="leg2" r="0" p="0" ry="${M_PI/2}" x="0" y="${bodyradius}"/>
 <xacro:leg leg="leg3" r="0" p="0" ry="${M_PI/6*5}" x="-${bodyradius/2*gen3}" y="${bodyradius/2}"/>
-<xacro:leg leg="leg4" r="0" p="0" ry="-${M_PI/6*5}" x="-${bodyradius/2*gen3}" y="-${bodyradius/2}"/>
+<xacro:leg leg="leg6" r="0" p="0" ry="-${M_PI/6*5}" x="-${bodyradius/2*gen3}" y="-${bodyradius/2}"/>
 <xacro:leg leg="leg5" r="0" p="0" ry="-${M_PI/2}" x="0" y="-${bodyradius}"/>
-<xacro:leg leg="leg6" r="0" p="0" ry="-${M_PI/6}" x="${bodyradius/2*gen3}" y="-${bodyradius/2}"/>
+<xacro:leg leg="leg4" r="0" p="0" ry="-${M_PI/6}" x="${bodyradius/2*gen3}" y="-${bodyradius/2}"/>
 </robot>
