Commit message: buffer模式调试完成版

File: src/hexapod_gazebo_description/urdf/hexapod_gazebo.xacro (robot description, xacro)
@@ -208,5 +208,5 @@
 <joint name="${leg}_pitch2" type="revolute">
   <axis xyz="0 0 1"/>
-  <limit effort="300" lower="-${M_PI/3}" upper="${M_PI/2}" velocity="1"/>
+  <limit effort="300" lower="-${M_PI/3}" upper="${M_PI*5/6}" velocity="1"/>
   <dynamics damping="${damping}"/>
   <parent link="${leg}_pitch1"/>
